File: oscilloscope_stm32F4/oscilloscope_stm32F4.sch (KiCad schematic (older format))
At the start: 21 parts, among them K1 AQY210EH, K2 AQY210EH, P2 CH_1, P5 CH_2, U1 STM32F411CEU6_-_UFQFPN48, U2 MCP6S21-I_SN, U3 MCP6S21-I_SN, U4 REF2033AIDDCR

Commit message: atualização
Parts:
- removed C1, C5: 30pF var, symbol Device:C_Variable
- removed C2, C4, C6: 100nF, symbol Device:C
- removed C3, C7: 47pF, symbol Device:C
- removed D1, D2: BAV99, Package_TO_SOT_SMD:SOT-23, symbol Diode:BAV99
- removed K1, K2: AQY210EH, DIP762W47P254L478H340Q4N, symbol ocilloscope_lib:AQY210EH
- removed P2: CH_1, symbol Connector:Conn_Coaxial
- removed P5: CH_2, symbol Connector:Conn_Coaxial
- removed R2, R6: 910K, symbol Device:R_US
- removed R3, R7: 100K, symbol Device:R_US
- removed U1: STM32F411CEU6_-_UFQFPN48, Package_DFN_QFN:QFN-48-1EP_7x7mm_P0.5mm_EP5.6x5.6mm, symbol ocilloscope_lib:STM32F411CEU6_-_UFQFPN48
- removed U2, U3: MCP6S21-I_SN, SOIC127P600X175-8N, symbol ocilloscope_lib:MCP6S21-I_SN
- removed U4: REF2033AIDDCR, DDC0005A_N, symbol ocilloscope_lib:REF2033AIDDCR
Connections:
- net labels removed: +3.3V, +5V, C14, GND, PA2, PGND
- wire segments 73 -> 0

Commit message: Atualizando...
Parts:
- added C1, C16: 30pF var, symbol Device:C_Variable
- added C10, C12: 12pF, symbol Device:C_Small
- added C11: 47uF, symbol Device:C_Small
- added C13: 2.2uF, symbol Device:C_Small
- added C14, C18: 47pF, symbol Device:C
- added C15, C17: 100nF, symbol Device:C
- added C19: C_Small, symbol Device:C_Small
- added C2, C3, C4, C5, C7: 100n, Capacitor_SMD:C_0805_2012Metric_Pad1.18x1.45mm_HandSolder, symbol Device:C
- added C6, C8: 10u, Capacitor_SMD:C_1210_3225Metric_Pad1.33x2.70mm_HandSolder, symbol Device:C
- added C9: 470nF, symbol Device:C_Small
- added D1, D2: BAV99, Package_TO_SOT_SMD:SOT-23, symbol Diode:BAV99
- added IC1: AMS1117-1.2, SOT229P700X180-4N, symbol ocilloscope_lib:AMS1117-1.2
- added J1: SW, Connector_PinSocket_2.54mm:PinSocket_1x04_P2.54mm_Vertical, symbol Connector:Conn_01x04_Male
- added J2: USB_B_Micro, Connector_USB:USB_Micro-B_Amphenol_10103594-0001LF_Horizontal, symbol Connector:USB_B_Micro
- added K1, K2: AQY210EH, DIP762W47P254L478H340Q4N, symbol ocilloscope_lib:AQY210EH
- added L1: 10uH ±10%, symbol pspice:INDUCTOR
- added P2: CH_1, symbol Connector:Conn_Coaxial
- added P5: CH_2, symbol Connector:Conn_Coaxial
- added R10: 1K, symbol Device:R_Small_US
- added R11: R_Small, symbol Device:R_Small
- added R2, R6: 910K, symbol Device:R_US
- added R3, R7: 100K, symbol Device:R_US
- added R8, R9: 10, symbol Device:R_Small
- added RV1: 1K, symbol Device:R_POT_US
- added SW1: SW_MEC_5E, symbol Switch:SW_MEC_5E
- added U1: STM32F411CEU6_-_UFQFPN48, Package_DFN_QFN:QFN-48-1EP_7x7mm_P0.5mm_EP5.6x5.6mm, symbol ocilloscope_lib:STM32F411CEU6_-_UFQFPN48
- added U2, U3: MCP6S21-I_SN, SOIC127P600X175-8N, symbol ocilloscope_lib:MCP6S21-I_SN
- added U4: LM1117-3.3, Package_TO_SOT_SMD:SOT-223-3_TabPin2, symbol Regulator_Linear:LM1117-3.3
- added Y2: 25MHz 9PF, symbol Device:Crystal_Small
Connections:
- new net: J1.2 (Pin_2), U1.34 (PA13)
- new net: J1.3 (Pin_3), U1.37 (PA14)
- new net: J2.2 (D-), R9.1
- new net: J2.3 (D+), R8.1
- new net: R8.2, U1.33 (PA12)
- new net: R9.2, U1.32 (PA11)
- new net: U1.13 (PA3), U2.1 (VOUT)
- new net: U1.15 (PA5), U3.1 (VOUT)
- new net: U1.39 (PB3), U2.7 (SCK), U3.7 (SCK)
- new net: U1.40 (PB4), U2.6 (SI), U3.6 (SI)
- new net: U1.41 (PB5), U2.5 (~CS)
- new net: U1.42 (PB6), U3.5 (~CS)
- new net: L1.2, U1.9 (VDDA)
- new net: C1.1, C14.1, D1.3 (K), R2.1, R3.1, U2.2 (CH0)
- new net: C15.2, K1.3, P2.1 (In)
- new net: C1.2, C15.1, K1.4, R2.2
- new net: C11.1, IC1.1 (GND/ADJUST), R10.2, RV1.1
- new net: C16.1, C18.1, D2.3 (K), R6.1, R7.1, U3.2 (CH0)
- new net: C17.2, K2.3, P5.1 (In)
- new net: C16.2, C17.1, K2.4, R6.2
- new net +3V3: C2.1, C3.1, C4.1, C5.1, C8.1, D1.2 (A), D2.2 (A), IC1.3 (VIN), J1.1 (Pin_1), L1.1, R11.2, U1.24 (VDD), U1.36 (VDD), U1.48 (VDD), U2.8 (VDD), U3.8 (VDD), U4.2 (VO)
- new net +5V: C6.1, C7.1, J2.1 (VBUS), U4.3 (VI)
- new net C14: K1.1, U1.3 (PC14)
- new net C15: K2.1, U1.4 (PC15)
- new net GND: C10.1, C11.2, C12.1, C13.2, C19.1, C2.2, C3.2, C4.2, C5.2, C6.2, C7.2, C8.2, C9.2, D1.1 (K), D2.1 (K), J1.4 (Pin_4), J2.4 (ID), J2.5 (GND), J2.6 (Shield), K1.2, K2.2, RV1.2, SW1.3 (K), SW1.4 (A), U1.23 (VSS), U1.35 (VSS), U1.47 (VSS), U1.8 (VSSA), U2.4 (VSS), U3.4 (VSS), U4.1 (GND)
- new net NRST: C19.2, R11.1, SW1.1, SW1.2, U1.7 (NRST)
- new net PGND: C14.2, C18.2, C9.1, IC1.2 (VOUT), P2.2 (Ext), P5.2 (Ext), R10.1, R3.2, R7.2, U2.3 (VREF), U3.3 (VREF)
- new net PH0: C12.2, U1.5 (PH0), Y2.2
- new net PH1: C10.2, U1.6 (PH1), Y2.1
- new net VCAP1: C13.1, U1.22 (VCAP1)
- no-connect marks 0 -> 27

Commit message: atualização
Parts:
- removed L1: 10uH ±10%, symbol pspice:INDUCTOR
- added C20, C22: 100n, Capacitor_SMD:C_0805_2012Metric_Pad1.18x1.45mm_HandSolder, symbol Device:C
- added C21: 4.7uF, symbol Device:C_Small
- added L1: 10uH, symbol Device:L_Small
- C19: value C_Small -> 0.1uF
- K1, K2: Description photomos relay 350V AQY210EH -> AC/DC SELECTOR
- R11: value R_Small -> 10k
Connections:
- net +3V3: now also C20.1, C21.1, C22.1, L1.2
- net GND: now also C20.2, C21.2, C22.2
- net SWDIO: now reaches J1.2 (Pin_2), U1.34 (PA13)
- net SWCLK: now reaches J1.3 (Pin_3), U1.37 (PA14)
- net USB_FS_DM: now reaches J2.2 (D-), R9.1
- net USB_FS_DP: now reaches J2.3 (D+), R8.1
- net PA12: now reaches R8.2, U1.33 (PA12)
- net PA11: now reaches R9.2, U1.32 (PA11)
- net Analog_CH-1: now reaches U1.13 (PA3), U2.1 (VOUT)
- net Analog_CH-2: now reaches U1.15 (PA5), U3.1 (VOUT)
- net at U1.9 (VDDA): now also L1.1
Other:
- moved on the sheet: C11, C13, C19, C2, C3, C4, C5, C9, IC1, J1, J2, R10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

Commit message: atualização
Parts:
- removed C21: 4.7uF, symbol Device:C_Small
- removed L1: 10uH, symbol Device:L_Small
- removed Y2: 25MHz 9PF, symbol Device:Crystal_Small
- added Y2: 25MHz 9PF, footprints:CrystalSMD, symbol Device:Crystal_GND24_Small
- C1, C16: footprint (none) -> footprints:JZ300
- C10, C12, C14, C18: footprint (none) -> Capacitor_SMD:C_0603_1608Metric_Pad1.08x0.95mm_HandSolder
- C11: footprint (none) -> Capacitor_Tantalum_SMD:CP_EIA-7132-20_AVX-U
- C13: value 2.2uF -> 4.7uF; footprint (none) -> Capacitor_SMD:C_0805_2012Metric_Pad1.18x1.45mm_HandSolder
- C15, C17, C19: footprint (none) -> Capacitor_SMD:C_0805_2012Metric_Pad1.18x1.45mm_HandSolder
- C22: value 100n -> 1uF
- C5: value 100n -> 4.7uF
- C9: footprint (none) -> footprints:CAPC1005X55N
- IC1: footprint SOT229P700X180-4N -> footprints:SOT229P700X180-4N
- K1, K2: footprint DIP762W47P254L478H340Q4N -> footprints:DIP762W47P254L478H340Q4N
- P2, P5: footprint (none) -> Connector_Coaxial:BNC_Amphenol_B6252HB-NPP3G-50_Horizontal
- R10, R11, R8, R9: footprint (none) -> Resistor_THT:R_Axial_DIN0204_L3.6mm_D1.6mm_P5.08mm_Horizontal
- R2, R6: footprint (none) -> Resistor_SMD:R_1210_3225Metric_Pad1.30x2.65mm_HandSolder
- R3, R7: footprint (none) -> Resistor_SMD:R_2512_6332Metric_Pad1.40x3.35mm_HandSolder
- RV1: footprint (none) -> Potentiometer_THT:Potentiometer_Bourns_3266Y_Vertical
- SW1: footprint (none) -> Button_Switch_SMD:SW_SPST_Omron_B3FS-100xP
- U2, U3: footprint SOIC127P600X175-8N -> footprints:SOIC127P600X175-8N
Connections:
- net +3V3: now also U1.1 (VBAT), U1.9 (VDDA)
- net PH0: now also Y2.1
- net PH1: now also Y2.3
- no-connect marks 27 -> 26
Other:
- moved on the sheet: C2, C20, C22, C3, C4, C5
