File: oscilloscope_stm32F4/oscilloscope_stm32F4.kicad_pcb (KiCad board)
At the start: 2 copper layers, 45 parts, among them IC1 AMS1117-1.2, J1 SW, J2 USB_B_Micro, K1 AQY210EH, K2 AQY210EH, P2 CH_1, P5 CH_2, SW1 SW_MEC_5E, U1 STM32F411CEU6_-_UFQFPN48, U2 MCP6S21-I_SN, U3 MCP6S21-I_SN, U4 LM1117-3.3, Y2 25MHz 9PF

Commit message: att
Parts:
- moved J1 27.5 mm to (114.3, 100.3), turned to 90 degrees
- moved C12 2.13 mm to (136.4, 90.9)
- moved R9 0.25 mm to (146.3, 88.6)
Routing:
- net VDD: track 34.7 -> 103.7 mm, vias 0 -> 3
- net C14: track 0.00 -> 33.7 mm, vias 0 -> 2
- net C15: track 33.3 -> 65.7 mm, vias 0 -> 1
- net /Analog_CH-2: track 0.00 -> 27.4 mm, vias 0 -> 2
- net GND: track 106.0 -> 132.0 mm, vias 11 -> 14
- net NRST: track 15.9 -> 39.9 mm
- net /Analog_CH-1: track 0.00 -> 23.0 mm, vias 0 -> 2
- net /SWDIO: track 0.00 -> 14.3 mm, vias 0 -> 2
- net Net-(U1-Pad41): track 0.00 -> 12.9 mm
- net Net-(U1-Pad40): track 0.00 -> 11.3 mm
- net /SWCLK: track 0.00 -> 10.8 mm, vias 0 -> 2
- net Net-(U1-Pad39): track 0.00 -> 9.78 mm
- net Net-(U1-Pad42): track 0.00 -> 9.26 mm, vias 0 -> 2
- net /PGND: track 35.2 -> 37.8 mm, vias 9 -> 11
- net PA12: track 23.5 -> 25.5 mm
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